Commit message: fixed odom math, working efk for imu and odom

File: src/robby_description/urdf/Robby_v1.core.xacro (robot description, xacro)
@@ -116,6 +116,7 @@
     <xacro:property name="back_right_wheel_rpy" value="-1.5708 0 -0.0078748" />
     <xacro:property name="front_right_wheel_rpy" value="-1.5708 0 -0.0087292" />
-    <xacro:mesh_box_link
-      name="base_link"
+    <link name="base_link" />
+    <xacro:mesh_box_link
+      name="chassis_link"
       inertial_xyz="-0.0202853583615552 -0.0035672102008257 0.0384224210186663"
       mass="2.2668069894461"
@@ -131,4 +132,9 @@
       collision_size="0.480668 0.396114 0.150001"
       mesh_uri_root="${mesh_uri_root}" />
+    <joint name="base_to_chassis_joint" type="fixed">
+      <origin xyz="0 0 0" rpy="0 0 0" />
+      <parent link="base_link" />
+      <child link="chassis_link" />
+    </joint>
     <link name="imu_link">
       <inertial>
@@ -140,5 +146,5 @@
     <joint name="imu_joint" type="fixed">
       <origin xyz="0 0 0.08" rpy="0 0 0" />
-      <parent link="base_link" />
+      <parent link="chassis_link" />
       <child link="imu_link" />
     </joint>
@@ -161,5 +167,5 @@
       name="f_left_steer"
       xyz="${front_left_steer_xyz}"
-      parent="base_link"
+      parent="chassis_link"
       child="front_left_steer"
       limit="${front_steer_limit}"
@@ -213,5 +219,5 @@
       name="b_leftsteer"
       xyz="${back_left_steer_xyz}"
-      parent="base_link"
+      parent="chassis_link"
       child="back_left_steer"
       limit="${rear_steer_limit}"
@@ -265,5 +271,5 @@
       name="b_rightsteer"
       xyz="${back_right_steer_xyz}"
-      parent="base_link"
+      parent="chassis_link"
       child="back_right_steer"
       limit="${rear_steer_limit}"
@@ -317,5 +323,5 @@
       name="f_right_steer"
       xyz="${front_right_steer_xyz}"
-      parent="base_link"
+      parent="chassis_link"
       child="front_right_steer"
       limit="${front_steer_limit}"

Commit message: implemented working kinamatic contoller layer

File: src/robby_description/urdf/Robby_v1.core.xacro (robot description, xacro)
@@ -88,5 +88,5 @@
     <xacro:property name="mesh_uri_root" value="file://${mesh_dir}" />
     <xacro:property name="front_steer_limit" value="1.5708" />
-    <xacro:property name="rear_steer_limit" value="0.0" />
+    <xacro:property name="rear_steer_limit" value="1.5708" />
     <xacro:property name="joint_effort" value="10" />
     <xacro:property name="joint_velocity" value="10" />

Commit message: Added Lidar and Camera sensors and also implemented slam tool box

File: src/robby_description/urdf/Robby_v1.core.xacro (robot description, xacro)
@@ -116,5 +116,12 @@
     <xacro:property name="back_right_wheel_rpy" value="-1.5708 0 -0.0078748" />
     <xacro:property name="front_right_wheel_rpy" value="-1.5708 0 -0.0087292" />
+    <xacro:property name="base_footprint_to_base_link_z" value="0.1478" />
+    <link name="base_footprint" />
     <link name="base_link" />
+    <joint name="base_footprint_joint" type="fixed">
+      <origin xyz="0 0 ${base_footprint_to_base_link_z}" rpy="0 0 0" />
+      <parent link="base_footprint" />
+      <child link="base_link" />
+    </joint>
     <xacro:mesh_box_link
       name="chassis_link"

File: src/robby_description/urdf/Robby_v1.gazebo.xacro (robot description, xacro)
@@ -4,5 +4,17 @@
   <xacro:arg name="controllers_file" default="" />
   <xacro:arg name="imu_update_rate" default="100.0" />
+  <xacro:arg name="use_lidar" default="false" />
+  <xacro:arg name="lidar_xyz" default="0 0 0.15" />
+  <xacro:arg name="lidar_rpy" default="0 0 0" />
+  <xacro:arg name="lidar_topic" default="/scan" />
+  <xacro:arg name="lidar_update_rate" default="15.0" />
+  <xacro:arg name="use_camera" default="false" />
+  <xacro:arg name="camera_xyz" default="0.12 0 0.18" />
+  <xacro:arg name="camera_rpy" default="0 0 0" />
+  <xacro:arg name="camera_topic" default="/camera/image_raw" />
+  <xacro:arg name="camera_update_rate" default="15.0" />
   <xacro:include filename="Robby_v1.core.xacro" />
+  <xacro:include filename="Robby_v1.lidar.xacro" />
+  <xacro:include filename="Robby_v1.camera.xacro" />
   <xacro:macro name="ros2_control_position_joint" params="joint_name">
     <joint name="${joint_name}">
@@ -20,4 +32,22 @@
   </xacro:macro>
   <xacro:robby_robot mesh_dir="$(arg mesh_dir)" />
+  <xacro:if value="$(arg use_lidar)">
+    <xacro:robby_lidar
+      parent="chassis_link"
+      xyz="$(arg lidar_xyz)"
+      rpy="$(arg lidar_rpy)"
+      add_gazebo="true"
+      topic="$(arg lidar_topic)"
+      update_rate="$(arg lidar_update_rate)" />
+  </xacro:if>
+  <xacro:if value="$(arg use_camera)">
+    <xacro:robby_camera
+      parent="chassis_link"
+      xyz="$(arg camera_xyz)"
+      rpy="$(arg camera_rpy)"
+      add_gazebo="true"
+      topic="$(arg camera_topic)"
+      update_rate="$(arg camera_update_rate)" />
+  </xacro:if>
   <gazebo reference="imu_link">
     <sensor name="imu_sensor" type="imu">
@@ -46,5 +76,5 @@
       <dimensions>2</dimensions>
       <odom_frame>ground_truth</odom_frame>
-      <robot_base_frame>base_link</robot_base_frame>
+      <robot_base_frame>base_footprint</robot_base_frame>
       <odom_topic>/ground_truth/odom</odom_topic>
       <gaussian_noise>0.0</gaussian_noise>

File: src/robby_description/urdf/Robby_v1.urdf.xacro (robot description, xacro)
@@ -3,5 +3,27 @@
 <robot xmlns:xacro="http://www.ros.org/wiki/xacro" name="Robby_v1">
   <xacro:arg name="mesh_dir" default="/home/aditya/ros2_ws/ITQ_robby/src/robby_description/meshes" />
+  <xacro:arg name="use_lidar" default="false" />
+  <xacro:arg name="lidar_xyz" default="0 0 0.15" />
+  <xacro:arg name="lidar_rpy" default="0 0 0" />
+  <xacro:arg name="use_camera" default="false" />
+  <xacro:arg name="camera_xyz" default="0.12 0 0.18" />
+  <xacro:arg name="camera_rpy" default="0 0 0" />
   <xacro:include filename="Robby_v1.core.xacro" />
+  <xacro:include filename="Robby_v1.lidar.xacro" />
+  <xacro:include filename="Robby_v1.camera.xacro" />
   <xacro:robby_robot mesh_dir="$(arg mesh_dir)" />
+  <xacro:if value="$(arg use_lidar)">
+    <xacro:robby_lidar
+      parent="chassis_link"
+      xyz="$(arg lidar_xyz)"
+      rpy="$(arg lidar_rpy)"
+      add_gazebo="false" />
+  </xacro:if>
+  <xacro:if value="$(arg use_camera)">
+    <xacro:robby_camera
+      parent="chassis_link"
+      xyz="$(arg camera_xyz)"
+      rpy="$(arg camera_rpy)"
+      add_gazebo="false" />
+  </xacro:if>
 </robot>

Commit message: updated the mesh from absilut path referance to a package referance

File: src/robby_description/urdf/Robby_v1.core.xacro (robot description, xacro)
@@ -86,5 +86,5 @@
   </xacro:macro>
   <xacro:macro name="robby_robot" params="mesh_dir">
-    <xacro:property name="mesh_uri_root" value="file://${mesh_dir}" />
+    <xacro:property name="mesh_uri_root" value="${mesh_dir}" />
     <xacro:property name="front_steer_limit" value="1.5708" />
     <xacro:property name="rear_steer_limit" value="1.5708" />

File: src/robby_description/urdf/Robby_v1.gazebo.xacro (robot description, xacro)
@@ -1,5 +1,5 @@
 <?xml version="1.0" encoding="utf-8"?>
 <robot xmlns:xacro="http://www.ros.org/wiki/xacro" name="Robby_v1">
-  <xacro:arg name="mesh_dir" default="/home/aditya/ros2_ws/ITQ_robby/src/robby_description/meshes" />
+  <xacro:arg name="mesh_dir" default="package://robby_description/meshes" />
   <xacro:arg name="controllers_file" default="" />
   <xacro:arg name="imu_update_rate" default="100.0" />

File: src/robby_description/urdf/Robby_v1.urdf.xacro (robot description, xacro)
@@ -2,5 +2,5 @@
 <!-- Clean robot description only. Gazebo and ros2_control live in Robby_v1.gazebo.xacro. -->
 <robot xmlns:xacro="http://www.ros.org/wiki/xacro" name="Robby_v1">
-  <xacro:arg name="mesh_dir" default="/home/aditya/ros2_ws/ITQ_robby/src/robby_description/meshes" />
+  <xacro:arg name="mesh_dir" default="package://robby_description/meshes" />
   <xacro:arg name="use_lidar" default="false" />
   <xacro:arg name="lidar_xyz" default="0 0 0.15" />
