Commit message: added camera module to the robot, needs working

File: src/robby_description/urdf/Robby_v1.camera.xacro (robot description, xacro)
@@ -5,8 +5,8 @@
     params="
       parent:=chassis_link
-      xyz:='0.12 0 0.18'
+      xyz:='0.15 0.0 0.0195'
       rpy:='0 0 0'
       add_gazebo:=false
-      topic:=/camera/image_raw
+      topic:=/camera
       update_rate:=15.0
       width:=640
@@ -18,14 +18,20 @@
       <inertial>
         <origin xyz="0 0 0" rpy="0 0 0" />
-        <mass value="0.12" />
-        <inertia ixx="8e-5" ixy="0.0" ixz="0.0" iyy="8e-5" iyz="0.0" izz="8e-5" />
+        <mass value="0.0387416202428435" />
+        <inertia
+          ixx="1.08456634317136E-05"
+          ixy="0.0"
+          ixz="0.0"
+          iyy="7.10436611069618E-06"
+          iyz="0.0"
+          izz="7.1103467824982E-06" />
       </inertial>
       <visual>
         <origin xyz="0 0 0" rpy="0 0 0" />
         <geometry>
-          <box size="0.05 0.04 0.035" />
+          <mesh filename="package://robby_description/meshes/camera_link.STL" />
         </geometry>
-        <material name="camera_black">
-          <color rgba="0.08 0.08 0.08 1.0" />
+        <material name="camera_body">
+          <color rgba="0.05 0.12 0.55 1" />
         </material>
       </visual>
@@ -33,5 +39,5 @@
         <origin xyz="0 0 0" rpy="0 0 0" />
         <geometry>
-          <box size="0.05 0.04 0.035" />
+          <box size="0.023 0.0421 0.0420" />
         </geometry>
       </collision>
@@ -56,5 +62,6 @@
     <xacro:if value="${add_gazebo}">
       <gazebo reference="camera_link">
-        <sensor name="camera_sensor" type="camera">
+        <material>Gazebo/Blue</material>
+        <sensor name="camera_sensor" type="rgbd_camera">
           <always_on>1</always_on>
           <update_rate>${update_rate}</update_rate>

File: src/robby_description/urdf/Robby_v1.gazebo.xacro (robot description, xacro)
@@ -5,13 +5,5 @@
   <xacro:arg name="imu_update_rate" default="100.0" />
   <xacro:arg name="use_lidar" default="false" />
-  <xacro:arg name="lidar_xyz" default="0 0 0.15" />
-  <xacro:arg name="lidar_rpy" default="0 0 0" />
-  <xacro:arg name="lidar_topic" default="/scan" />
-  <xacro:arg name="lidar_update_rate" default="15.0" />
   <xacro:arg name="use_camera" default="false" />
-  <xacro:arg name="camera_xyz" default="0.12 0 0.18" />
-  <xacro:arg name="camera_rpy" default="0 0 0" />
-  <xacro:arg name="camera_topic" default="/camera/image_raw" />
-  <xacro:arg name="camera_update_rate" default="15.0" />
   <xacro:include filename="Robby_v1.core.xacro" />
   <xacro:include filename="Robby_v1.lidar.xacro" />
@@ -33,20 +25,8 @@
   <xacro:robby_robot mesh_dir="$(arg mesh_dir)" />
   <xacro:if value="$(arg use_lidar)">
-    <xacro:robby_lidar
-      parent="chassis_link"
-      xyz="$(arg lidar_xyz)"
-      rpy="$(arg lidar_rpy)"
-      add_gazebo="true"
-      topic="$(arg lidar_topic)"
-      update_rate="$(arg lidar_update_rate)" />
+    <xacro:robby_lidar add_gazebo="true" />
   </xacro:if>
   <xacro:if value="$(arg use_camera)">
-    <xacro:robby_camera
-      parent="chassis_link"
-      xyz="$(arg camera_xyz)"
-      rpy="$(arg camera_rpy)"
-      add_gazebo="true"
-      topic="$(arg camera_topic)"
-      update_rate="$(arg camera_update_rate)" />
+    <xacro:robby_camera add_gazebo="true" />
   </xacro:if>
   <gazebo reference="imu_link">

File: src/robby_description/urdf/Robby_v1.urdf.xacro (robot description, xacro)
@@ -4,9 +4,5 @@
   <xacro:arg name="mesh_dir" default="package://robby_description/meshes" />
   <xacro:arg name="use_lidar" default="false" />
-  <xacro:arg name="lidar_xyz" default="0 0 0.15" />
-  <xacro:arg name="lidar_rpy" default="0 0 0" />
   <xacro:arg name="use_camera" default="false" />
-  <xacro:arg name="camera_xyz" default="0.12 0 0.18" />
-  <xacro:arg name="camera_rpy" default="0 0 0" />
   <xacro:include filename="Robby_v1.core.xacro" />
   <xacro:include filename="Robby_v1.lidar.xacro" />
@@ -14,16 +10,8 @@
   <xacro:robby_robot mesh_dir="$(arg mesh_dir)" />
   <xacro:if value="$(arg use_lidar)">
-    <xacro:robby_lidar
-      parent="chassis_link"
-      xyz="$(arg lidar_xyz)"
-      rpy="$(arg lidar_rpy)"
-      add_gazebo="false" />
+    <xacro:robby_lidar add_gazebo="false" />
   </xacro:if>
   <xacro:if value="$(arg use_camera)">
-    <xacro:robby_camera
-      parent="chassis_link"
-      xyz="$(arg camera_xyz)"
-      rpy="$(arg camera_rpy)"
-      add_gazebo="false" />
+    <xacro:robby_camera add_gazebo="false" />
   </xacro:if>
 </robot>
